File: board/board.kicad_sch (KiCad schematic)
At the start: 1 part

Commit message: initial
Parts:
- removed LOGO1: Logo_Open_Hardware_Small, Symbol:OSHW-Symbol_6.7x6mm_SilkScreen, symbol Graphic:Logo_Open_Hardware_Small
- added J1: Conn_01x10_Male, on_edge:on_edge_2x05_device, symbol Connector:Conn_01x10_Male
- added J2, J3, J4, J5: Conn_01x05_Male, Connector_PinSocket_2.54mm:PinSocket_1x05_P2.54mm_Vertical, symbol Connector:Conn_01x05_Male
- added J6: Conn_01x10_Male, on_edge:on_edge_2x05_host, symbol Connector:Conn_01x10_Male
Connections:
- new net: J1.1 (Pin_1), J2.1 (Pin_1)
- new net: J1.10 (Pin_10), J3.5 (Pin_5)
- new net: J1.2 (Pin_2), J2.2 (Pin_2)
- new net: J1.3 (Pin_3), J2.3 (Pin_3)
- new net: J1.4 (Pin_4), J2.4 (Pin_4)
- new net: J1.5 (Pin_5), J2.5 (Pin_5)
- new net: J1.6 (Pin_6), J3.1 (Pin_1)
- new net: J1.7 (Pin_7), J3.2 (Pin_2)
- new net: J1.8 (Pin_8), J3.3 (Pin_3)
- new net: J1.9 (Pin_9), J3.4 (Pin_4)
- new net: J4.1 (Pin_1), J6.1 (Pin_1)
- new net: J4.2 (Pin_2), J6.2 (Pin_2)
- new net: J4.3 (Pin_3), J6.3 (Pin_3)
- new net: J4.4 (Pin_4), J6.4 (Pin_4)
- new net: J4.5 (Pin_5), J6.5 (Pin_5)
- new net: J5.1 (Pin_1), J6.6 (Pin_6)
- new net: J5.2 (Pin_2), J6.7 (Pin_7)
- new net: J5.3 (Pin_3), J6.8 (Pin_8)
- new net: J5.4 (Pin_4), J6.9 (Pin_9)
- new net: J5.5 (Pin_5), J6.10 (Pin_10)
Other:
- removed sheet implementation
- note removed: "Input connectors go here"
- note removed: "Output connectors go here"
Changed lines of the file:
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@@
 (kicad_sch (version 20211123) (generator eeschema)
   (paper "A4")
-  (text "Output connectors go here" (at 224.79 88.9 0)
-    (effects (font (size 1.27 1.27)) (justify left bottom))
+  (wire (pts (xy 167.64 92.075) (xy 158.75 92.075))
+    (stroke (width 0) (type default) (color 0 0 0 0))
   )
-  (text "Input connectors go here" (at 49.53 88.9 0)
-    (effects (font (size 1.27 1.27)) (justify left bottom))
+  (wire (pts (xy 146.05 112.395) (xy 134.62 112.395))
+    (stroke (width 0) (type default) (color 0 0 0 0))
   )
-  (symbol (lib_id "Graphic:Logo_Open_Hardware_Small") (at 273.05 157.48 0) (unit 1)
-    (in_bom yes) (on_board yes) (fields_autoplaced)
-    (property "Reference" "LOGO1" (id 0) (at 273.05 150.495 0)
+  (wire (pts (xy 167.64 102.235) (xy 158.75 102.235))
+    (stroke (width 0) (type default) (color 0 0 0 0))
+  )
+  (wire (pts (xy 167.64 107.315) (xy 158.75 107.315))
+    (stroke (width 0) (type default) (color 0 0 0 0))
+  )
+  (wire (pts (xy 146.05 92.075) (xy 134.62 92.075))
+    (stroke (width 0) (type default) (color 0 0 0 0))
+  )
+  (wire (pts (xy 167.64 89.535) (xy 158.75 89.535))
+    (stroke (width 0) (type default) (color 0 0 0 0))
+  )
+  (wire (pts (xy 146.05 89.535) (xy 134.62 89.535))
+    (stroke (width 0) (type default) (color 0 0 0 0))
+  )
+  (wire (pts (xy 146.05 102.235) (xy 134.62 102.235))
+    (stroke (width 0) (type default) (color 0 0 0 0))
+  )
+  (wire (pts (xy 167.64 99.695) (xy 158.75 99.695))
+    (stroke (width 0) (type default) (color 0 0 0 0))
+  )
+  (wire (pts (xy 167.64 97.155) (xy 158.75 97.155))
+    (stroke (width 0) (type default) (color 0 0 0 0))
+  )
+  (wire (pts (xy 167.64 94.615) (xy 158.75 94.615))
+    (stroke (width 0) (type default) (color 0 0 0 0))
+  )
+  (wire (pts (xy 167.64 109.855) (xy 158.75 109.855))
+    (stroke (width 0) (type default) (color 0 0 0 0))
+  )
+  (wire (pts (xy 146.05 109.855) (xy 134.62 109.855))
+    (stroke (width 0) (type default) (color 0 0 0 0))
+  )
+  (wire (pts (xy 146.05 107.315) (xy 134.62 107.315))
+    (stroke (width 0) (type default) (color 0 0 0 0))
+  )
+  (wire (pts (xy 146.05 97.155) (xy 134.62 97.155))
+    (stroke (width 0) (type default) (color 0 0 0 0))
+  )
+  (wire (pts (xy 146.05 104.775) (xy 134.62 104.775))
+    (stroke (width 0) (type default) (color 0 0 0 0))
+  )
+  (wire (pts (xy 167.64 112.395) (xy 158.75 112.395))
+    (stroke (width 0) (type default) (color 0 0 0 0))
+  )
+  (wire (pts (xy 146.05 99.695) (xy 134.62 99.695))
+    (stroke (width 0) (type default) (color 0 0 0 0))
+  )
+  (wire (pts (xy 167.64 104.775) (xy 158.75 104.775))
+    (stroke (width 0) (type default) (color 0 0 0 0))
+  )
+  (wire (pts (xy 146.05 94.615) (xy 134.62 94.615))
+    (stroke (width 0) (type default) (color 0 0 0 0))
+  )
+  (symbol (lib_id "Connector:Conn_01x10_Male") (at 139.7 99.695 0) (mirror y) (unit 1)
+    (in_bom yes) (on_board yes)
+    (property "Reference" "J1" (id 0) (at 136.9568 84.9376 0))
+    (property "Value" "Conn_01x10_Male" (id 1) (at 136.9568 87.249 0))
+    (property "Footprint" "on_edge:on_edge_2x05_device" (id 2) (at 139.7 99.695 0)
       (effects (font (size 1.27 1.27)) hide)
     )
-    (property "Value" "Logo_Open_Hardware_Small" (id 1) (at 273.05 163.195 0)
+    (property "Datasheet" "~" (id 3) (at 139.7 99.695 0)
       (effects (font (size 1.27 1.27)) hide)
     )
-    (property "Footprint" "Symbol:OSHW-Symbol_6.7x6mm_SilkScreen" (id 2) (at 273.05 157.48 0)
+    (pin "1")
+    (pin "10")
+    (pin "2")
+    (pin "3")
+    (pin "4")
+    (pin "5")
+    (pin "6")
+    (pin "7")
+    (pin "8")
+    (pin "9")
+  )
+  (symbol (lib_id "Connector:Conn_01x05_Male") (at 163.83 94.615 0) (mirror y) (unit 1)
+    (in_bom yes) (on_board yes)
+    (property "Reference" "J4" (id 0) (at 161.0868 84.9376 0))
+    (property "Value" "Conn_01x05_Male" (id 1) (at 161.0868 87.249 0))
+    (property "Footprint" "Connector_PinSocket_2.54mm:PinSocket_1x05_P2.54mm_Vertical" (id 2) (at 163.83 94.615 0)
       (effects (font (size 1.27 1.27)) hide)
     )
-    (property "Datasheet" "~" (id 3) (at 273.05 157.48 0)
+    (property "Datasheet" "~" (id 3) (at 163.83 94.615 0)
       (effects (font (size 1.27 1.27)) hide)
     )
+    (pin "1")
+    (pin "2")
+    (pin "3")
+    (pin "4")
+    (pin "5")
   )
-  (sheet (at 114.3 72.39) (size 60.96 62.23) (fields_autoplaced)
-    (stroke (width 0.1524) (type solid) (color 0 0 0 0))
-    (fill (color 0 0 0 0.0000))
-    (property "Sheet name" "implementation" (id 0) (at 114.3 71.6784 0)
-      (effects (font (size 1.27 1.27)) (justify left bottom))
+  (symbol (lib_id "Connector:Conn_01x05_Male") (at 151.13 94.615 0) (mirror y) (unit 1)
+    (in_bom yes) (on_board yes)
+    (property "Reference" "J2" (id 0) (at 148.3868 84.9376 0))
+    (property "Value" "Conn_01x05_Male" (id 1) (at 148.3868 87.249 0))
+    (property "Footprint" "Connector_PinSocket_2.54mm:PinSocket_1x05_P2.54mm_Vertical" (id 2) (at 151.13 94.615 0)
+      (effects (font (size 1.27 1.27)) hide)
     )
-    (property "Sheet file" "implementation.kicad_sch" (id 1) (at 114.3 135.2046 0)
-      (effects (font (size 1.27 1.27)) (justify left top))
+    (property "Datasheet" "~" (id 3) (at 151.13 94.615 0)
+      (effects (font (size 1.27 1.27)) hide)
     )
+    (pin "1")
+    (pin "2")
+    (pin "3")
+    (pin "4")
+    (pin "5")
+  )
+  (symbol (lib_id "Connector:Conn_01x05_Male") (at 151.13 107.315 0) (mirror y) (unit 1)
+    (in_bom yes) (on_board yes)
+    (property "Reference" "J3" (id 0) (at 148.3868 97.6376 0))
+    (property "Value" "Conn_01x05_Male" (id 1) (at 148.3868 99.949 0))
+    (property "Footprint" "Connector_PinSocket_2.54mm:PinSocket_1x05_P2.54mm_Vertical" (id 2) (at 151.13 107.315 0)
+      (effects (font (size 1.27 1.27)) hide)
+    )
+    (property "Datasheet" "~" (id 3) (at 151.13 107.315 0)
+      (effects (font (size 1.27 1.27)) hide)
+    )
+    (pin "1")
+    (pin "2")
+    (pin "3")
+    (pin "4")
+    (pin "5")
+  )
+  (symbol (lib_id "Connector:Conn_01x05_Male") (at 163.83 107.315 0) (mirror y) (unit 1)
+    (in_bom yes) (on_board yes)
+    (property "Reference" "J5" (id 0) (at 161.0868 97.6376 0))
+    (property "Value" "Conn_01x05_Male" (id 1) (at 161.0868 99.949 0))
+    (property "Footprint" "Connector_PinSocket_2.54mm:PinSocket_1x05_P2.54mm_Vertical" (id 2) (at 163.83 107.315 0)
+      (effects (font (size 1.27 1.27)) hide)
+    )
+    (property "Datasheet" "~" (id 3) (at 163.83 107.315 0)
+      (effects (font (size 1.27 1.27)) hide)
+    )
+    (pin "1")
+    (pin "2")
+    (pin "3")
+    (pin "4")
+    (pin "5")
+  )
+  (symbol (lib_id "Connector:Conn_01x10_Male") (at 172.72 99.695 0) (mirror y) (unit 1)
+    (in_bom yes) (on_board yes)
+    (property "Reference" "J6" (id 0) (at 169.9768 84.9376 0))
+    (property "Value" "Conn_01x10_Male" (id 1) (at 169.9768 87.249 0))
+    (property "Footprint" "on_edge:on_edge_2x05_host" (id 2) (at 172.72 99.695 0)
+      (effects (font (size 1.27 1.27)) hide)
+    )
+    (property "Datasheet" "~" (id 3) (at 172.72 99.695 0)
+      (effects (font (size 1.27 1.27)) hide)
+    )
+    (pin "1")
+    (pin "10")
+    (pin "2")
+    (pin "3")
+    (pin "4")
+    (pin "5")
+    (pin "6")
+    (pin "7")
+    (pin "8")
+    (pin "9")
   )
   (sheet_instances
     (path "/" (page "1"))
-    (path "/767ce4c6-0e55-4543-92f0-34cb8237a544" (page "2"))
   )
   (symbol_instances
-    (path "/b72b6f4a-7489-40f2-bb90-d75ae01aa368"
-      (reference "LOGO1") (unit 1) (value "Logo_Open_Hardware_Small") (footprint "Symbol:OSHW-Symbol_6.7x6mm_SilkScreen")
+    (path "/00000000-0000-0000-0000-0000602487d2"
+      (reference "J1") (unit 1) (value "Conn_01x10_Male") (footprint "on_edge:on_edge_2x05_device")
+    )
+    (path "/00000000-0000-0000-0000-000060252e83"
+      (reference "J2") (unit 1) (value "Conn_01x05_Male") (footprint "Connector_PinSocket_2.54mm:PinSocket_1x05_P2.54mm_Vertical")
+    )
+    (path "/00000000-0000-0000-0000-000060253690"
+      (reference "J3") (unit 1) (value "Conn_01x05_Male") (footprint "Connector_PinSocket_2.54mm:PinSocket_1x05_P2.54mm_Vertical")
+    )
+    (path "/00000000-0000-0000-0000-000060252352"
+      (reference "J4") (unit 1) (value "Conn_01x05_Male") (footprint "Connector_PinSocket_2.54mm:PinSocket_1x05_P2.54mm_Vertical")
+    )
+    (path "/00000000-0000-0000-0000-000060253dd5"
+      (reference "J5") (unit 1) (value "Conn_01x05_Male") (footprint "Connector_PinSocket_2.54mm:PinSocket_1x05_P2.54mm_Vertical")
+    )
+    (path "/00000000-0000-0000-0000-0000602592e9"
+      (reference "J6") (unit 1) (value "Conn_01x10_Male") (footprint "on_edge:on_edge_2x05_host")
     )
   )
